File: farlock3.kicad_sch (KiCad schematic)
At the start: 11 parts

Commit message: farlock3 v01 layout, production files
Parts:
- removed U?: MCP73831-2-OT, Package_TO_SOT_SMD:SOT-23-5, symbol Battery_Management:MCP73831-2-OT
- added C10, C11: 1.0µF, Capacitor_SMD:C_0603_1608Metric, symbol Device:C
- added C14, C15: 300pF, Capacitor_SMD:C_0603_1608Metric, symbol Device:C
- added C16: dnp, Capacitor_SMD:C_0603_1608Metric, symbol Device:C
- added C17: DNP, Capacitor_SMD:C_0603_1608Metric, symbol Device:C
- added C6, C7, C9: 0.1µF, Capacitor_SMD:C_0603_1608Metric, symbol Device:C
- added C8: 10µF, Capacitor_Tantalum_SMD:CP_EIA-3528-21_Kemet-B, symbol Device:C_Polarized_US
- added D1: Red, LED_SMD:LED_0603_1608Metric, symbol Device:LED
- added D2: 6A/45V/520mV, Package_TO_SOT_SMD:TO-277A, symbol Device:D_Schottky_Dual_CommonCathode_AAK_Parallel
- added D5: Blue, LED_SMD:LED_0603_1608Metric, symbol Device:LED
- added J2: Conn_01x17, Connector_PinHeader_2.54mm:PinHeader_1x17_P2.54mm_Vertical, symbol Connector_Generic:Conn_01x17
- added JP1: Power LED, Jumper:SolderJumper-2_P1.3mm_Bridged_RoundedPad1.0x1.5mm, symbol Jumper:SolderJumper_2_Bridged
- added JP2: NFC1, Jumper:SolderJumper-2_P1.3mm_Bridged_RoundedPad1.0x1.5mm, symbol Jumper:SolderJumper_2_Bridged
- added JP3: NFC2, Jumper:SolderJumper-2_P1.3mm_Bridged_RoundedPad1.0x1.5mm, symbol Jumper:SolderJumper_2_Bridged
- added JP4: NFC2, Jumper:SolderJumper-2_P1.3mm_Open_RoundedPad1.0x1.5mm, symbol Jumper:SolderJumper_2_Open
- added JP5: NFC1, Jumper:SolderJumper-2_P1.3mm_Open_RoundedPad1.0x1.5mm, symbol Jumper:SolderJumper_2_Open
- added R1, R2: 27, Resistor_SMD:R_0603_1608Metric, symbol Device:R_US
- added R3, R6: 1k, Resistor_SMD:R_0603_1608Metric, symbol Device:R_US
- added R7: 10k, Resistor_SMD:R_0603_1608Metric, symbol Device:R_US
- added R8, R9: 330, Resistor_SMD:R_0603_1608Metric, symbol Device:R_US
- added SW1: SW_SPDT, Button_Switch_SMD:SW_SPDT_PCM12, symbol Switch:SW_SPDT
- added U2: MX25R6435FZNIL0, Package_SON:WSON-8-1EP_6x5mm_P1.27mm_EP3.4x4mm, symbol MX25R6435F:MX25R6435FZNIL0
- C1, C2: renamed from C?; footprint (none) -> Capacitor_SMD:C_0603_1608Metric; Manufacturer Part No (none) -> CL10A106MP8NNNC
- C3: renamed from C?; footprint (none) -> Capacitor_SMD:C_0603_1608Metric; Manufacturer Part No (none) -> CL10B104KA8NNNC
- C4, C5: renamed from C?; footprint (none) -> Capacitor_SMD:C_0603_1608Metric; Manufacturer Part No (none) -> CL10C150JB8NNNC
- J1: renamed from J?; footprint (none) -> Connector_USB:USB_Micro-B_Amphenol_10104110_Horizontal; Manufacturer Part No (none) -> 10104110-0001LF
- U1: renamed from U?; footprint (none) -> MDBT50Q:MDBT50Q; Manufacturer Part No (none) -> MDBT50Q-U1MV2
- U3: renamed from U?; Manufacturer Part No (none) -> TB6612FNG,C,8,EL
- U4: renamed from U?; Manufacturer Part No (none) -> AP2112K-3.3TRG1
- Y1: renamed from Y?; footprint (none) -> Crystal:Crystal_SMD_3215-2Pin_3.2x1.5mm; Manufacturer Part No (none) -> CM7V-T1A-LOW-ESR-32.768KHZ-9PF-20-TA-QC
Connections:
- net GND: now also C1.2, C2.2, C3.2, C4.2, C5.2, J1.5 (GND), J1.6 (Shield), U1.1 (GND@1), U1.15 (GND@15), U1.2 (GND@2), U1.33 (GND@33), U1.55 (GND@55), U3.10 (PGND2), U3.18 (GND), U3.3 (PGND1), U3.4 (PGND1), U3.9 (PGND2), U4.2 (GND), C10.2, C11.2, C14.2, C15.2, C16.2, C17.2, C6.2, C7.2, C8.2, C9.2, J2.10 (Pin_10), J2.2 (Pin_2), JP1.1 (A), SW1.1 (A), U2.4 (GND)
- net P0.29: now reaches U1.10 (P0.29/AIN5)
- net P0.29: now also U3.21 (AIN1)
- net P0.31: now reaches U1.12 (P0.31/AIN7)
- net P0.31: now also U3.19 (STBY)
- net P0.28: now reaches U1.13 (P0.28/AIN4)
- net P0.28: now also U3.23 (PWMA)
- net P0.30: now reaches U1.14 (P0.30/AIN6)
- net P0.30: now also U3.22 (AIN2)
- net at U1.17 (P0.00/XL1): now also C4.1, Y1.1
- net at U1.18 (P0.01/XL2): now also C5.1, Y1.2
- net +3V3: now reaches U1.28 (VDD)
- net +3V3: now also C1.1, C2.1, C3.1, U1.30 (VDDH), U3.20 (VCC), U4.5 (VOUT), C11.1, C6.1, C9.1, J2.3 (Pin_3), J2.6 (Pin_6), R3.1, R6.1, R7.2, R8.1, R9.1, U2.8 (VCC)
- net VBUS: now reaches U1.32 (VBUS)
- net VBUS: now also J1.1 (VBUS), D2.2 (A)
- net at U1.34 (D-): now also R1.1
- net at U1.35 (D+): now also R2.1
- net P0.13: now reaches U1.37 (P0.13)
- net P0.13: now also D5.1 (K)
- net LED_ACCD-: now reaches U1.38 (P0.16)
- net LED_ACCD-: now also J2.12 (Pin_12)
- net LED_ACCG-: now reaches U1.39 (P0.15)
- net LED_ACCG-: now also J2.14 (Pin_14)
- net RESET: now reaches U1.40 (P0.18/RESET)
- net RESET: now also J2.9 (Pin_9)
- net P0.17: now reaches U1.41 (P0.17)
- net P0.17: now also U2.1 (~{CS})
- net P0.19: now reaches U1.42 (P0.19)
- net P0.19: now also U2.6 (SCLK)
- net P0.21: now reaches U1.43 (P0.21)
- net P0.21: now also U2.2 (SO/SIO1)
- net P0.20: now reaches U1.44 (P0.20)
- net P0.20: now also U2.5 (SI/SIO0)
- net P0.23: now reaches U1.45 (P0.23)
- net P0.23: now also U2.7 (~{RESET}/SIO3)
- net P0.22: now reaches U1.46 (P0.22)
- net P0.22: now also U2.3 (~{WP}/SIO2)
- net P0.25: now reaches U1.49 (P0.25)
- net P0.25: now also J2.11 (Pin_11), R7.1
- net SWDIO: now reaches U1.51 (SWDIO)
- net SWDIO: now also J2.7 (Pin_7)
- net P0.09/NFC1: now reaches U1.52 (P0.09/NFC1)
- net P0.09/NFC1: now also J2.17 (Pin_17), JP2.2 (B), JP5.2 (B)
- net SWDCLK: now reaches U1.53 (SWDCLK)
- net SWDCLK: now also J2.8 (Pin_8)
- net P0.10/NFC2: now reaches U1.54 (P0.10/NFC2)
- net P0.10/NFC2: now also J2.16 (Pin_16), JP3.2 (B), JP4.2 (B)
- net MOTOR_1: now reaches U3.1 (AO1), U3.2 (AO1)
- net MOTOR_1: now also J2.4 (Pin_4)
- net +VDC: now reaches U3.13 (VM2)
- net +VDC: now also U3.14 (VM3), U3.24 (VM1), U4.1 (VIN), C10.1, C7.1, C8.1, D2.3 (K), SW1.3 (C)
- net MOTOR_2: now reaches U3.5 (AO2), U3.6 (AO2)
- net MOTOR_2: now also J2.5 (Pin_5)
- net at U4.3 (EN): now also SW1.2 (B)
- net D-_CON: now reaches J1.2 (D-)
- net D-_CON: now also R1.2
- net D+_CON: now reaches J1.3 (D+)
- net D+_CON: now also R2.2
- new net: C16.1, JP5.1 (A)
- new net: D1.1 (K), JP1.2 (B)
- new net: D1.2 (A), R3.2
- new net: C17.1, JP4.1 (A)
- new net: C14.1, JP2.1 (A)
- new net: D5.2 (A), R6.2
- new net: C15.1, JP3.1 (A)
- new net LED_ACCD+: J2.13 (Pin_13), R9.2
- new net LED_ACCG+: J2.15 (Pin_15), R8.2
- new net VIN: D2.1 (A), J2.1 (Pin_1)
- no-connect marks 0 -> 38
Other:
- moved on the sheet: J1, U3, U4

Commit message: v02 redesign
Parts:
- removed J2: Conn_01x17, Connector_PinHeader_2.54mm:PinHeader_1x17_P2.54mm_Vertical, symbol Connector_Generic:Conn_01x17
- added C12: 10µF, Capacitor_SMD:C_0603_1608Metric, symbol Device:C
- added C13: 0.1µF, Capacitor_SMD:C_0603_1608Metric, symbol Device:C
- added D3: PRTR5V0U2X, Package_TO_SOT_SMD:SOT-143, symbol Power_Protection:PRTR5V0U2X
- added J2: Conn_01x05, Connector_PinHeader_2.54mm:PinHeader_1x05_P2.54mm_Vertical, symbol Connector_Generic:Conn_01x05
- added J3, J4: Conn_01x02, Connector_PinHeader_2.54mm:PinHeader_1x02_P2.54mm_Vertical, symbol Connector_Generic:Conn_01x02
- added J5: Conn_01x10, Connector_PinHeader_2.54mm:PinHeader_1x10_P2.54mm_Vertical, symbol Connector_Generic:Conn_01x10
- added J6: Conn_01x03, Connector_PinHeader_2.54mm:PinHeader_1x03_P2.54mm_Vertical, symbol Connector_Generic:Conn_01x03
- added R10: 330, Resistor_SMD:R_0603_1608Metric, symbol Device:R_US
- added R4, R5: 10k, Resistor_SMD:R_0603_1608Metric, symbol Device:R_US
- C16, C17: now not fitted
- SW1: footprint Button_Switch_SMD:SW_SPDT_PCM12 -> OS102011MA1QN1:OS102011MA1QN1; Manufacturer Part No PCM12SMTR -> OS102011MA1QN1
- U1: footprint MDBT50Q:MDBT50Q -> MDBT50Q:MDBT50Q-U1M
Connections:
- net +3V3: now also J2.5 (Pin_5), R10.1, R4.2, R5.2
- net +VDC: now also U4.3 (EN); no longer SW1.3 (C)
- net GND: now also SW1.3 (C), C12.2, C13.2, D3.1 (GND), J2.4 (Pin_4), J5.1 (Pin_1), J5.6 (Pin_6), J6.1 (Pin_1); no longer SW1.1 (A)
- net LED_ACCD+: now also J5.8 (Pin_8)
- net LED_ACCD-: now also J5.7 (Pin_7)
- net LED_ACCG+: now also J5.10 (Pin_10)
- net LED_ACCG-: now also J5.9 (Pin_9)
- net MOTOR_1: now also J5.4 (Pin_4)
- net MOTOR_2: now also J5.3 (Pin_3)
- net P0.09/NFC1: now also J4.2 (Pin_2)
- net P0.10/NFC2: now also J4.1 (Pin_1)
- net P0.25: now also J5.2 (Pin_2), R4.1; no longer R7.1
- net RESET: now also J2.3 (Pin_3)
- net SWDCLK: now also J2.2 (Pin_2)
- net SWDIO: now also J2.1 (Pin_1)
- net VBUS: now also C12.1, C13.1, D3.4 (VCC)
- net VIN: now also J5.5 (Pin_5)
- net P0.12: now reaches U1.29 (P0.12)
- net P0.12: now also J6.3 (Pin_3), R5.1
- net LED_CXN-: now reaches U1.36 (P0.14)
- net LED_CXN-: now also J3.1 (Pin_1)
- net P0.24: now reaches U1.48 (P0.24)
- net P0.24: now also R7.1, SW1.2 (B)
- net D+_CON renamed D+
- net D+: now also D3.3 (I/O2)
- net D-_CON renamed D-
- net D-: now also D3.2 (I/O1)
- new net LED_CXN+: J3.2 (Pin_2), R10.2
- no-connect marks 38 -> 35
Other:
- moved on the sheet: C10, C11, C14, C15, D1, D2, D5, J1, JP1, JP2, JP3, JP4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
